Commit message: Align BG2 rev4 follower hardware config

File: ffw_description/ros2_control/ffw_bg2_rev4_follower/ffw_bg2_follower.ros2_control.xacro (robot description, xacro)
@@ -20,11 +20,11 @@
             <param name="baud_rate">4000000</param>
             <param name="dynamixel_model_folder">/param/dxl_model</param>
-            <param name="number_of_joints">19</param>
-            <param name="number_of_transmissions">19</param>
+            <param name="number_of_joints">17</param>
+            <param name="number_of_transmissions">17</param>
             <param name="disable_torque_at_init">true</param>
-            <param name="dynamixel_state_pub_msg_name">ffw_follower/dxl_state</param>
-            <param name="get_dynamixel_data_srv_name">ffw_follower/get_dxl_data</param>
-            <param name="set_dynamixel_data_srv_name">ffw_follower/set_dxl_data</param>
-            <param name="reboot_dxl_srv_name">ffw_follower/reboot_dxl</param>
+            <param name="dynamixel_state_pub_msg_name">dynamixel_hardware_interface/dxl_state</param>
+            <param name="get_dynamixel_data_srv_name">dynamixel_hardware_interface/get_dxl_data</param>
+            <param name="set_dynamixel_data_srv_name">dynamixel_hardware_interface/set_dxl_data</param>
+            <param name="reboot_dxl_srv_name">dynamixel_hardware_interface/reboot_dxl</param>
             <param name="set_dxl_torque_srv_name">dynamixel_hardware_interface/set_dxl_torque</param>
           </xacro:unless>
@@ -73,10 +73,4 @@
         <state_interface name="effort"/>
       </joint>
-      <joint name="gripper_r_joint1">
-        <command_interface name="position"/>
-        <state_interface name="position"/>
-        <state_interface name="velocity"/>
-        <state_interface name="effort"/>
-      </joint>
       <joint name="arm_l_joint1">
         <command_interface name="position"/>
@@ -116,10 +110,4 @@
       </joint>
       <joint name="arm_l_joint7">
-        <command_interface name="position"/>
-        <state_interface name="position"/>
-        <state_interface name="velocity"/>
-        <state_interface name="effort"/>
-      </joint>
-      <joint name="gripper_l_joint1">
         <command_interface name="position"/>
         <state_interface name="position"/>
@@ -309,17 +297,4 @@
         <param name="Min Position Limit">-151875</param>
       </gpio>
-      <gpio name="dxl8">
-        <param name="type">dxl</param>
-        <param name="ID">8</param>
-        <command_interface name="Goal Position"/>
-        <state_interface name="Present Position"/>
-        <state_interface name="Present Velocity"/>
-        <state_interface name="Present Current"/>
-        <state_interface name="Hardware Error Status"/>
-        <param name="Operating Mode">5</param>
-        <param name="Return Delay Time">0</param>
-        <param name="Profile Velocity">0</param>
-        <param name="Profile Acceleration">0</param>
-      </gpio>
       <!-- LEFT ARM -->
       <gpio name="dxl31">
@@ -486,17 +461,4 @@
         <param name="Min Position Limit">-151875</param>
       </gpio>
-      <gpio name="dxl38">
-        <param name="type">dxl</param>
-        <param name="ID">38</param>
-        <command_interface name="Goal Position"/>
-        <state_interface name="Present Position"/>
-        <state_interface name="Present Velocity"/>
-        <state_interface name="Present Current"/>
-        <state_interface name="Hardware Error Status"/>
-        <param name="Operating Mode">5</param>
-        <param name="Return Delay Time">0</param>
-        <param name="Profile Velocity">0</param>
-        <param name="Profile Acceleration">0</param>
-      </gpio>
       <!-- LIFT -->
       <gpio name="dxl81">
@@ -543,5 +505,5 @@
         <param name="Profile Velocity">100</param>
         <param name="Profile Acceleration">50</param>
-        <param name="Max Position Limit">2560</param>
+        <param name="Max Position Limit">2500</param>
         <param name="Min Position Limit">1896</param>
         <param name="Position P Gain">1600</param>
