Commit message: Backup ai_worker_robot snapshot

File: ffw_description/ros2_control/ffw_bg2_rev4_follower/ffw_bg2_follower.ros2_control copy.xacro (robot description, xacro)
@@ -535,4 +535,25 @@
       </gpio>
     </ros2_control>
+    <xacro:unless value="$(arg use_sim)">
+      <ros2_control name="ffw_bg2_follower_fake_gripper" type="system">
+        <hardware>
+          <plugin>mock_components/GenericSystem</plugin>
+          <param name="mock_sensor_commands">false</param>
+          <param name="state_following_offset">0.0</param>
+        </hardware>
+        <joint name="gripper_r_joint1">
+          <command_interface name="position"/>
+          <state_interface name="position"/>
+          <state_interface name="velocity"/>
+          <state_interface name="effort"/>
+        </joint>
+        <joint name="gripper_l_joint1">
+          <command_interface name="position"/>
+          <state_interface name="position"/>
+          <state_interface name="velocity"/>
+          <state_interface name="effort"/>
+        </joint>
+      </ros2_control>
+    </xacro:unless>
   </xacro:macro>
 </robot>
